File: eimer/eimer.kicad_sch (KiCad schematic)
At the start: 71 parts, among them J3 Conn_01x03, J4 USB_C_Receptacle_USB2.0_14P, SW1 SW_Push, SW2 SW_Push, U1 RP2040, U2 MCP1700x-330xxTT, U3 TPS61221DCK, U4 W25Q16JVUXIQ TR, U5 LIS2DW12, Y1 12 MHz

Commit message: routing leds
Connections:
- net GPIO26/ADC0: now also R14.2; no longer TP1.1
- net GPIO27/ADC1: now also R15.2; no longer TP2.1
- net GPIO28/ADC2: now also R16.2; no longer TP3.1
- net GPIO29/ADC3: now also R17.2; no longer TP4.1
- net GPIO1: now reaches U1.3 (GPIO1)
- net GPIO1: now also R10.2
- net GPIO2: now reaches U1.4 (GPIO2)
- net GPIO2: now also R11.2
- net GPIO4: now reaches U1.6 (GPIO4)
- net GPIO4: now also R12.2
- net GPIO6: now reaches U1.8 (GPIO6)
- net GPIO6: now also R13.2
- net GPIO11: no longer names the net of U1.14 (GPIO11)
- net GPIO11: no longer R10.2
- net GPIO12: no longer names the net of U1.15 (GPIO12)
- net GPIO12: no longer R11.2
- net GPIO13: no longer names the net of U1.16 (GPIO13)
- net GPIO13: no longer R12.2
- net GPIO14: no longer names the net of U1.17 (GPIO14)
- net GPIO15: no longer names the net of U1.18 (GPIO15)
- net GPIO15: no longer R14.2
- net GPIO16: no longer names the net of U1.27 (GPIO16)
- net GPIO16: no longer R15.2
- net GPIO17: no longer names the net of U1.28 (GPIO17)
- net GPIO17: no longer R16.2
- net GPIO18: no longer names the net of U1.29 (GPIO18)
- net GPIO18: no longer R17.2
- net GPIO20: no longer names the net of U1.31 (GPIO20)
- net GPIO20: no longer TP5.1
- net GPIO22: no longer names the net of TP6.1
- net GPIO22: no longer U1.34 (GPIO22)
- net GPIO23: no longer names the net of U1.35 (GPIO23)
- net GPIO23: no longer TP7.1
- net GPIO24: no longer names the net of TP8.1
- net GPIO24: no longer U1.36 (GPIO24)
- no-connect marks 10 -> 4

Commit message: routed all left side gpios
Connections:
- net GPIO11: now reaches TP1.1
- net GPIO11: now also U1.14 (GPIO11)
- net GPIO13: now reaches TP3.1
- net GPIO13: now also U1.16 (GPIO13)
- net GPIO12: now reaches U1.15 (GPIO12)
- net GPIO12: now also TP2.1
- net GPIO15: now reaches U1.18 (GPIO15)
- net GPIO15: now also TP4.1
Changed lines of the file:
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@@
+		)
+	)
+	(global_label "GPIO11"
+		(shape bidirectional)
+		(at 254 207.01 0)
+		(fields_autoplaced yes)
+		(effects
+			(font
+				(size 1.27 1.27)
+			)
+			(justify left)
+		)
+		(property "Intersheetrefs" "${INTERSHEET_REFS}"
+			(at 264.9908 207.01 0)
+			(hide yes)
+			(show_name no)
+			(do_not_autoplace no)
+			(effects
+				(font
+					(size 1.27 1.27)
+				)
+				(justify left)
+			)
 		)
 	)
@@
 		)
 	)
+	(global_label "GPIO15"
+		(shape bidirectional)
+		(at 254 217.17 0)
+		(fields_autoplaced yes)
+		(effects
+			(font
+				(size 1.27 1.27)
+			)
+			(justify left)
+		)
+		(property "Intersheetrefs" "${INTERSHEET_REFS}"
+			(at 264.9908 217.17 0)
+			(hide yes)
+			(show_name no)
+			(do_not_autoplace no)
+			(effects
+				(font
+					(size 1.27 1.27)
+				)
+				(justify left)
+			)
+		)
+	)
+	(global_label "GPIO11"
+		(shape bidirectional)
+		(at 104.775 179.07 0)
+		(fields_autoplaced yes)
+		(effects
+			(font
+				(size 1.27 1.27)
+			)
+			(justify left)
+		)
+		(property "Intersheetrefs" "${INTERSHEET_REFS}"
+			(at 115.7658 179.07 0)
+			(hide yes)
+			(show_name no)
+			(do_not_autoplace no)
+			(effects
+				(font
+					(size 1.27 1.27)
+				)
+				(justify left)
+			)
+		)
+	)
 	(global_label "XOUT"
 		(shape output)
@@
 		)
 	)
+	(global_label "GPIO12"
+		(shape bidirectional)
+		(at 104.775 186.69 0)
+		(fields_autoplaced yes)
+		(effects
+			(font
+				(size 1.27 1.27)
+			)
+			(justify left)
+		)
+		(property "Intersheetrefs" "${INTERSHEET_REFS}"
+			(at 115.7658 186.69 0)
+			(hide yes)
+			(show_name no)
+			(do_not_autoplace no)
+			(effects
+				(font
+					(size 1.27 1.27)
+				)
+				(justify left)
+			)
+		)
+	)
 	(global_label "USB_D-"
 		(shape bidirectional)
@@
 		)
 	)
+	(global_label "GPIO15"
+		(shape bidirectional)
+		(at 104.775 201.93 0)
+		(fields_autoplaced yes)
+		(effects
+			(font
+				(size 1.27 1.27)
+			)
+			(justify left)
+		)
+		(property "Intersheetrefs" "${INTERSHEET_REFS}"
+			(at 115.7658 201.93 0)
+			(hide yes)
+			(show_name no)
+			(do_not_autoplace no)
+			(effects
+				(font
+					(size 1.27 1.27)
+				)
+				(justify left)
+			)
+		)
+	)
+	(global_label "GPIO12"
+		(shape bidirectional)
+		(at 254 209.55 0)
+		(fields_autoplaced yes)
+		(effects
+			(font
+				(size 1.27 1.27)
+			)
+			(justify left)
+		)
+		(property "Intersheetrefs" "${INTERSHEET_REFS}"
+			(at 264.9908 209.55 0)
+			(hide yes)
+			(show_name no)
+			(do_not_autoplace no)
+			(effects
+				(font
+					(size 1.27 1.27)
+				)
+				(justify left)
+			)
+		)
+	)
 	(global_label "USB_D+"
 		(shape bidirectional)
@@
 		(property "Intersheetrefs" "${INTERSHEET_REFS}"
 			(at 77.4844 240.665 0)
+			(hide yes)
+			(show_name no)
+			(do_not_autoplace no)
+			(effects
+				(font
+					(size 1.27 1.27)
+				)
+				(justify left)
+			)
+		)
+	)
+	(global_label "GPIO13"
+		(shape bidirectional)
+		(at 104.775 194.31 0)
+		(fields_autoplaced yes)
+		(effects
+			(font
+				(size 1.27 1.27)
+			)
+			(justify left)
+		)
+		(property "Intersheetrefs" "${INTERSHEET_REFS}"
+			(at 115.7658 194.31 0)
 			(hide yes)
 			(show_name no)
@@
 			(hide yes)
 			(show_name no)
+			(do_not_autoplace no)
+			(effects
+				(font
+					(size 1.27 1.27)
+				)
+				(justify left)
+			)
+		)
+	)
+	(global_label "GPIO13"
+		(shape bidirectional)
+		(at 254 212.09 0)
+		(fields_autoplaced yes)
+		(effects
+			(font
+				(size 1.27 1.27)
+			)
+			(justify left)
+		)
+		(property "Intersheetrefs" "${INTERSHEET_REFS}"
+			(at 264.9908 212.09 0)
+			(hide yes)
+			(show_name no)

Commit message: routed all gpios
Connections:
- net GPIO21: now reaches TP8.1
- net GPIO21: now also U1.32 (GPIO21)
- net GPIO19: now reaches TP6.1
- net GPIO19: now also U1.30 (GPIO19)
- net GPIO18: now reaches U1.29 (GPIO18)
- net GPIO18: now also TP5.1
- net GPIO20: now reaches U1.31 (GPIO20)
- net GPIO20: now also TP7.1
- no-connect marks 4 -> 1
Changed lines of the file:
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@@
 	)
 	(no_connect
-		(at 252.73 242.57)
-	)
-	(no_connect
-		(at 254 227.33)
-	)
-	(no_connect
 		(at 254 196.85)
 	)
-	(no_connect
-		(at 254 232.41)
-	)
 	(wire
 		(pts
@@
 		)
 	)
+	(global_label "GPIO18"
+		(shape bidirectional)
+		(at 254 224.79 0)
+		(fields_autoplaced yes)
+		(effects
+			(font
+				(size 1.27 1.27)
+			)
+			(justify left)
+		)
+		(property "Intersheetrefs" "${INTERSHEET_REFS}"
+			(at 264.9908 224.79 0)
+			(hide yes)
+			(show_name no)
+			(do_not_autoplace no)
+			(effects
+				(font
+					(size 1.27 1.27)
+				)
+				(justify left)
+			)
+		)
+	)
 	(global_label "INT2"
 		(shape bidirectional)
@@
 		)
 	)
+	(global_label "GPIO19"
+		(shape bidirectional)
+		(at 254 227.33 0)
+		(fields_autoplaced yes)
+		(effects
+			(font
+				(size 1.27 1.27)
+			)
+			(justify left)
+		)
+		(property "Intersheetrefs" "${INTERSHEET_REFS}"
+			(at 264.9908 227.33 0)
+			(hide yes)
+			(show_name no)
+			(do_not_autoplace no)
+			(effects
+				(font
+					(size 1.27 1.27)
+				)
+				(justify left)
+			)
+		)
+	)
 	(global_label "XIN"
 		(shape output)
@@
 		)
 	)
+	(global_label "GPIO20"
+		(shape bidirectional)
+		(at 254 229.87 0)
+		(fields_autoplaced yes)
+		(effects
+			(font
+				(size 1.27 1.27)
+			)
+			(justify left)
+		)
+		(property "Intersheetrefs" "${INTERSHEET_REFS}"
+			(at 264.9908 229.87 0)
+			(hide yes)
+			(show_name no)
+			(do_not_autoplace no)
+			(effects
+				(font
+					(size 1.27 1.27)
+				)
+				(justify left)
+			)
+		)
+	)
 	(global_label "GPIO28{slash}ADC2"
 		(shape bidirectional)
@@
 		)
 	)
+	(global_label "GPIO19"
+		(shape bidirectional)
+		(at 104.775 218.44 0)
+		(fields_autoplaced yes)
+		(effects
+			(font
+				(size 1.27 1.27)
+			)
+			(justify left)
+		)
+		(property "Intersheetrefs" "${INTERSHEET_REFS}"
+			(at 115.7658 218.44 0)
+			(hide yes)
+			(show_name no)
+			(do_not_autoplace no)
+			(effects
+				(font
+					(size 1.27 1.27)
+				)
+				(justify left)
+			)
+		)
+	)
 	(global_label "GPIO12"
 		(shape bidirectional)
@@
 		)
 	)
+	(global_label "GPIO20"
+		(shape bidirectional)
+		(at 104.775 226.06 0)
+		(fields_autoplaced yes)
+		(effects
+			(font
+				(size 1.27 1.27)
+			)
+			(justify left)
+		)
+		(property "Intersheetrefs" "${INTERSHEET_REFS}"
+			(at 115.7658 226.06 0)
+			(hide yes)
+			(show_name no)
+			(do_not_autoplace no)
+			(effects
+				(font
+					(size 1.27 1.27)
+				)
+				(justify left)
+			)
+		)
+	)
 	(global_label "QSPI_SD2"
 		(shape bidirectional)
@@
 		)
 	)
+	(global_label "GPIO18"
+		(shape bidirectional)
+		(at 104.775 210.82 0)
+		(fields_autoplaced yes)
+		(effects
+			(font
+				(size 1.27 1.27)
+			)
+			(justify left)
+		)
+		(property "Intersheetrefs" "${INTERSHEET_REFS}"
+			(at 115.7658 210.82 0)
+			(hide yes)
+			(show_name no)
+			(do_not_autoplace no)
+			(effects
+				(font
+					(size 1.27 1.27)
+				)
+				(justify left)
+			)
+		)
+	)
 	(global_label "GPIO12"
 		(shape bidirectional)
@@
 		)
 	)
+	(global_label "GPIO21"
+		(shape bidirectional)
+		(at 104.775 233.68 0)
+		(fields_autoplaced yes)
+		(effects
+			(font
+				(size 1.27 1.27)
+			)
+			(justify left)
+		)
+		(property "Intersheetrefs" "${INTERSHEET_REFS}"
+			(at 115.7658 233.68 0)
+			(hide yes)
+			(show_name no)
+			(do_not_autoplace no)
+			(effects
+				(font
+					(size 1.27 1.27)
+				)
+				(justify left)
+			)
+		)
+	)
 	(global_label "GPIO1"
 		(shape input)
@@
 			(hide yes)
 			(show_name no)
+			(do_not_autoplace no)
+			(effects
+				(font
+					(size 1.27 1.27)
+				)
+				(justify left)
+			)
+		)
+	)
+	(global_label "GPIO21"
+		(shape bidirectional)
+		(at 253.9318 232.41 0)
+		(fields_autoplaced yes)
+		(effects
+			(font
+				(size 1.27 1.27)
+			)
+			(justify left)
+		)
+		(property "Intersheetrefs" "${INTERSHEET_REFS}"
+			(at 264.9226 232.41 0)
+			(hide yes)
+			(show_name no)

Commit message: removed some silkscreen text
Connections:
- no-connect marks 1 -> 10
Changed lines of the file:
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@@
+	)
+	(no_connect
+		(at 254 219.71)
+	)
+	(no_connect
+		(at 254 242.57)
 	)
 	(no_connect
 		(at 254 196.85)
 	)
+	(no_connect
+		(at 254 240.03)
+	)
+	(no_connect
+		(at 254 222.25)
+	)
+	(no_connect
+		(at 254 234.95)
+	)
+	(no_connect
+		(at 254 237.49)
+	)
+	(no_connect
+		(at 254 214.63)
+	)
+	(no_connect
+		(at 254 179.07)
+	)
+	(no_connect
+		(at 254 186.69)
+	)
 	(wire
 		(pts
@@
 		)
 		(stroke
+			(width 0)
+			(type default)
+		)
+	)
+	(wire
+		(pts
+			(xy 252.73 242.57) (xy 254 242.57)
+		)
+		(stroke
